File: KiCAD/ESP32 Sensing.kicad_pcb (KiCad board)
At the start: 2 copper layers, 29.9 x 27.9 mm, 34 parts, among them J2 Ext Battery 3.3V, J3 Sensor, J4 Thermistor, J5 Light Detect, J6 MICRO-B USB, Q1 MMBT3904, Q2 NDS356AP, SW1 PTS526_SK15_SMTR2_LFS, U1 ESP32-WROOM-32, U2 AMS1117-3.3

Commit message: Modified linear regulator  capacitor values
Parts:
- C2, C5: value 10n -> 10u
Changed lines of the file:
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@@
   (net 43 "Net-(D2-Pad1)")
   (net 44 "Net-(D3-Pad2)")
-  (net 45 "Net-(R3-Pad2)")
+  (net 45 "Net-(Q2-Pad3)")
   (footprint "Connector_PinHeader_2.54mm:PinHeader_1x02_P2.54mm_Vertical" (layer "F.Cu")
     (at 119.239515 104.601318)
@@
       (net 8 "A2D") (pintype "passive"))
     (pad "2" smd roundrect (at 1 0 270) (size 1.2 1.4) (layers "B.Cu" "B.Paste" "B.Mask") (roundrect_rratio 0.2083333333)
-      (net 45 "Net-(R3-Pad2)") (pintype "passive"))
+      (net 45 "Net-(Q2-Pad3)") (pintype "passive"))
     (model "${KICAD6_3DMODEL_DIR}/Resistor_SMD.3dshapes/R_0805_2012Metric.wrl"
       (offset (xyz 0 0 0))
@@
       (effects (font (size 1 1) (thickness 0.15)) (justify mirror))
     )
-    (fp_text value "10n" (at 0 -1.68 90) (layer "B.Fab") hide
+    (fp_text value "10u" (at 0 -1.68 90) (layer "B.Fab") hide
       (effects (font (size 1 1) (thickness 0.15)) (justify mirror))
     )
@@
       (net 5 "+3V3") (pinfunction "S") (pintype "passive"))
     (pad "3" smd roundrect (at 0.9375 0 90) (size 1.475 0.6) (layers "B.Cu" "B.Paste" "B.Mask") (roundrect_rratio 0.25)
-      (net 45 "Net-(R3-Pad2)") (pinfunction "D") (pintype "passive"))
+      (net 45 "Net-(Q2-Pad3)") (pinfunction "D") (pintype "passive"))
     (model "${KICAD6_3DMODEL_DIR}/Package_TO_SOT_SMD.3dshapes/SOT-23.wrl"
       (offset (xyz 0 0 0))
@@
       (effects (font (size 1 1) (thickness 0.15)) (justify mirror))
     )
-    (fp_text value "10n" (at 0 -1.68 90) (layer "B.Fab") hide
-      (effects (font (size 1 1) (thickness 0.15)) (justify mirror))
-    )
+    (fp_text value "10u" (at 0 -1.68 90) (layer "B.Fab") hide
+      (effects (font (size 1 1) (thickness 0.15)) (justify mirror))
+    )

Commit message: Version 2.0
Parts:
- added D4: LED, LED_SMD:LED_0805_2012Metric_Pad1.15x1.40mm_HandSolder, F.Cu at (119.5, 120.7)
- added J7: Conn_01x04_Male, Connector_PinHeader_2.54mm:PinHeader_1x04_P2.54mm_Vertical, F.Cu at (119.3, 110.2)
- added R14: 3K3, Resistor_SMD:R_0805_2012Metric_Pad1.20x1.40mm_HandSolder, B.Cu at (118.6, 121.2)
- added R15: 3K3, Resistor_SMD:R_0805_2012Metric_Pad1.20x1.40mm_HandSolder, B.Cu at (122.8, 117.0)
- added R16: 220, Resistor_SMD:R_0805_2012Metric_Pad1.20x1.40mm_HandSolder, B.Cu at (121.8, 121.2)
- C1, R6: moved to B.Cu
- R1: value 10k -> 2M7
- moved C1 12.8 mm to (127.9, 121.5), turned to -90 degrees
- moved REF** 11.6 mm to (132.3, 112.7)
- moved R6 8.42 mm to (125.8, 121.5)
- moved D3 7.84 mm to (119.5, 123.2), turned to 0 degrees
- moved SW2 3.95 mm to (125.8, 120.2), turned to -90 degrees
- moved R12 2.85 mm to (122.9, 112.6)
- moved Q2 2.43 mm to (129.3, 108.2)
- moved Q1 2.31 mm to (127.6, 115.9)
- moved R13 1.95 mm to (134.2, 121.8), turned to -90 degrees
- moved D1 1.04 mm to (143.8, 119.2), turned to 90 degrees
- moved D2 0.84 mm to (139.9, 102.9), turned to 90 degrees
- moved R5 0.75 mm to (137.5, 116.0), turned to -90 degrees
- moved J6 0.59 mm to (134.0, 121.2)
- moved J5 0.56 mm to (119.3, 104.0)
- moved J2 0.10 mm to (119.3, 97.8)
Connections:
- J4 pad 2: GPIO25 -> GPIO34
- J5 pad 2: GPIO27 -> GPIO35
- R11 pad 2: GPIO25 -> GPIO34
- R12 pad 2: GPIO27 -> GPIO35
- R8 pad 2: GPIO15 -> GPIO32
- R9 pad 2: GPIO15 -> GPIO32
- U1 pad 10: GPIO25 -> unconnected-(U1-Pad10)
- U1 pad 12: GPIO27 -> unconnected-(U1-Pad12)
- U1 pad 14: unconnected-(U1-Pad14) -> GPIO12
- U1 pad 23: GPIO15 -> unconnected-(U1-Pad23)
- U1 pad 33: unconnected-(U1-Pad33) -> SDA
- U1 pad 36: unconnected-(U1-Pad36) -> SCL
- U1 pad 6: unconnected-(U1-Pad6) -> GPIO34
- U1 pad 7: unconnected-(U1-Pad7) -> GPIO35
- U1 pad 8: unconnected-(U1-Pad8) -> GPIO32
Routing:
- net SCL: track 0.00 -> 49.0 mm, vias 0 -> 1
- net SDA: track 0.00 -> 40.2 mm, vias 0 -> 3
- net GPIO34: track 0.00 -> 29.7 mm, vias 0 -> 1
- net GPIO25: track 28.4 -> 0.00 mm, vias 1 -> 0
- net GPIO32: track 0.00 -> 27.3 mm, vias 0 -> 4
- net GND: track 2.22 -> 23.1 mm, vias 8 -> 9
- net GPIO27: track 16.4 -> 0.00 mm
- net GPIO15: track 14.7 -> 0.00 mm, vias 3 -> 0
- net GPIO35: track 0.00 -> 13.6 mm
- net +3V3: track 74.0 -> 84.0 mm
- net Net-(D3-Pad2): track 6.95 -> 14.2 mm
- net GPIO12: track 0.00 -> 6.78 mm, vias 0 -> 1
- net Net-(Q1-Pad1): track 12.0 -> 5.89 mm
- net Net-(Q1-Pad3): track 12.0 -> 8.75 mm
- net Net-(Q2-Pad3): track 5.04 -> 8.17 mm
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Other:
- board size 29.9 x 27.9 mm -> 29.9 x 28.6 mm
- board text added: "A"
- board text added: "D"
- board text added: "ESP32 SENSING V2.0"
- board text added: "Guy Turcotte - May 2022"
- board text removed: "ESP32 SENSING V1.0"
- board text removed: "Guy Turcotte - March 2022"
