File: V1.0 Files/KiCAD/ESP32 Sensing.kicad_sch (KiCad schematic)
At the start: 38 parts, among them J2 Ext Battery 3.3V, J3 Sensor, J4 Thermistor, J5 Light Detect, J6 MICRO-B USB, J7 Conn_01x04_Male, Q1 MMBT3904, Q2 NDS356AP, SW1 PTS526_SK15_SMTR2_LFS, U1 ESP32-WROOM-32, U2 AMS1117-3.3

Commit message: Version 2.0
Parts:
- removed D4: LED, LED_SMD:LED_0805_2012Metric_Pad1.15x1.40mm_HandSolder, symbol Device:LED
- removed J7: Conn_01x04_Male, Connector_PinHeader_2.54mm:PinHeader_1x04_P2.54mm_Vertical, symbol Connector:Conn_01x04_Male
- removed R14, R15: 3K3, Resistor_SMD:R_0805_2012Metric_Pad1.20x1.40mm_HandSolder, symbol Device:R
- removed R16: 220, Resistor_SMD:R_0805_2012Metric_Pad1.20x1.40mm_HandSolder, symbol Device:R
- C2: value 10u -> (none); footprint Capacitor_SMD:C_0805_2012Metric_Pad1.18x1.45mm_HandSolder -> (none)
- C5: value 10u -> (none)
- R1: value 2M7 -> 10k
Connections:
- net GPIO25: now reaches U1.10 (IO25)
- net GPIO25: now also J4.2 (Pin_2), R11.2
- net GPIO27: now reaches U1.12 (IO27)
- net GPIO27: now also J5.2 (Pin_2), R12.2
- net GPIO15: now reaches U1.23 (IO15)
- net GPIO15: now also R8.2, R9.2
- net GPIO12: no longer names the net of U1.14 (IO12)
- removed net GPIO32: R8.2, R9.2, U1.8 (IO32)
- removed net GPIO34: J4.2 (Pin_2), R11.2, U1.6 (IO34)
- removed net GPIO35: J5.2 (Pin_2), R12.2, U1.7 (IO35)
- net SCL: no longer names the net of U1.36 (IO22)
- net SDA: no longer names the net of U1.33 (IO21)
Other:
- note removed: "I2C"
- note removed: "PGM LED"
